File: IMU_BARO/Sensors/Sensors.kicad_pcb (KiCad board)
At the start: 2 copper layers, 50 x 50 mm, 26 parts, among them J1 Conn_02x02_Odd_Even, J2 Conn_02x05_Odd_Even, J3 Conn_02x04_Odd_Even, U1 LSM6DSV32XTR, U3 LSM303AGR, U5 BMP585

Commit message: Auto commit: 2025-02-26_20-32
Routing:
- net GND: vias 19 -> 251
- added copper zone on F.Cu, net GND
