File: PWM/pwm_servo/pwm_servo.kicad_pcb (KiCad board)
At the start: 4 copper layers, 50 x 50 mm, 30 parts, among them J1 Conn_01x03_MountingPin, J10 Conn_02x04_Odd_Even, J2 Conn_01x03_MountingPin, J3 Conn_01x03_MountingPin, J4 Conn_01x03_MountingPin, J5 Conn_02x04_Odd_Even, J6 Conn_02x04_Odd_Even, J7 Conn_02x04_Odd_Even, J8 Conn_02x04_Odd_Even, J9 Conn_02x04_Odd_Even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

Commit message: Auto commit: 2025-02-26_20-32
Routing:
- net GND: vias 1 -> 152
