File: brain_board/brain_board.kicad_pcb (KiCad board)
At the start: 6 copper layers, 50 x 50 mm, 58 parts, among them IC2 W25N01GVZEIG, J1 503398-1892, J10 Conn_02x05_Odd_Even, J2 USB_C_Receptacle_USB2.0_16P, J3 Conn_01x06_MountingPin, J4 Conn_02x04_Odd_Even, J5 Conn_02x04_Odd_Even, J6 Conn_02x04_Odd_Even, J7 Conn_02x04_Odd_Even, J8 Conn_02x02_Odd_Even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

Commit message: Auto commit: 2025-02-26_20-32
Parts:
- added J11: Conn_01x04_MountingPin, Connector_JST:JST_GH_SM04B-GHS-TB_1x04-1MP_P1.25mm_Horizontal, B.Cu at (134.3, 88.8)
- added J12: Conn_01x04_MountingPin, Connector_JST:JST_GH_SM04B-GHS-TB_1x04-1MP_P1.25mm_Horizontal, B.Cu at (134.3, 98.5)
Connections:
- U1 pad 22: unconnected-(U1-PA0-Pad22) -> /UART4_TX
- U1 pad 23: unconnected-(U1-PA1-Pad23) -> /UART4_RX
- U1 pad 37: unconnected-(U1-PE7-Pad37) -> /UART7_RX
- U1 pad 38: unconnected-(U1-PE8-Pad38) -> /UART7_TX
Routing:
- net +3.3V: track 70.8 -> 93.3 mm, vias 57 -> 63
- net /UART7_TX: track 0.00 -> 8.75 mm, vias 0 -> 1
- net /UART7_RX: track 0.00 -> 8.02 mm, vias 0 -> 1
- net /UART4_RX: track 0.00 -> 6.80 mm, vias 0 -> 1
- net /UART4_TX: track 0.00 -> 4.84 mm, vias 0 -> 1
- net GND: track 41.4 -> 45.6 mm, vias 76 -> 174
- added copper zone on In2.Cu, net GND
Other:
- board text added: "3v3"
- board text added: "GND"
- board text added: "RX"
- board text added: "TX"
