File: brain_board/brain_board.kicad_sch (KiCad schematic)
At the start: 58 parts, among them IC2 W25N01GVZEIG, J1 503398-1892, J10 Conn_02x05_Odd_Even, J2 USB_C_Receptacle_USB2.0_16P, J3 Conn_01x06_MountingPin, J4 Conn_02x04_Odd_Even, J5 Conn_02x04_Odd_Even, J6 Conn_02x04_Odd_Even, J7 Conn_02x04_Odd_Even, J8 Conn_02x02_Odd_Even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

Commit message: Auto commit: 2025-02-26_20-32
Parts:
- added J11, J12: Conn_01x04_MountingPin, Connector_JST:JST_GH_SM04B-GHS-TB_1x04-1MP_P1.25mm_Horizontal, symbol Connector_Generic_MountingPin:Conn_01x04_MountingPin
Connections:
- net +3.3V: now also J11.4 (Pin_4), J12.4 (Pin_4)
- net GND: now also J11.1 (Pin_1), J12.1 (Pin_1)
- net UART4_TX: now reaches U1.22 (PA0)
- net UART4_TX: now also J11.3 (Pin_3)
- net UART4_RX: now reaches U1.23 (PA1)
- net UART4_RX: now also J11.2 (Pin_2)
- net UART7_RX: now reaches U1.37 (PE7)
- net UART7_RX: now also J12.3 (Pin_3)
- net UART7_TX: now reaches U1.38 (PE8)
- net UART7_TX: now also J12.2 (Pin_2)
- no-connect marks 5 -> 7
